Commit message: using action service

File: src/abb_gofa_description/urdf/abb_gofa/abb_gofa_ros2_control.urdf.xacro (robot description, xacro)
@@ -5,5 +5,5 @@
         <!-- ===== Gazebo ROS2_CONTROL plugin ===== -->
         <gazebo>
-            <!-- <plugin name="link_attacher_plugin" filename="liblink_attacher_plugin.so"></plugin> -->
+            <plugin name="link_attacher_plugin" filename="liblink_attacher_plugin.so"></plugin>
             <plugin filename="libgazebo_ros2_control.so" name="gazebo_ros2_control">
                 <robot_sim_type>gazebo_ros2_control/GazeboSystem</robot_sim_type>

File: src/abb_gofa_description/urdf/egp64/egp64.urdf.xacro (robot description, xacro)
@@ -6,6 +6,6 @@
         <inertial>
             <origin xyz="0.0 0.0 0.0" rpy="0.0 0.0 0.0"/>
-            <mass value="0.5" />
-            <inertia ixx="0.00" ixy="0.0" ixz="0.0" iyy="0.00" iyz="0.0" izz="0.00"/>
+            <mass value="0.001" />
+            <inertia ixx="0.001" ixy="0.0" ixz="0.0" iyy="0.001" iyz="0.0" izz="0.001"/>
         </inertial>
         <visual>
@@ -38,6 +38,6 @@
         <inertial>
         <origin xyz="0 0 0" rpy="0 0 ${pi/2}" />
-        <mass value="0.1" />
-        <inertia ixx="0.00" ixy="0.0" ixz="0.0" iyy="0.000" iyz="0.0" izz="0.000"/>
+        <mass value="0.001" />
+        <inertia ixx="0.001" ixy="0.0" ixz="0.0" iyy="0.001" iyz="0.0" izz="0.001"/>
         </inertial>
     </link>
@@ -50,6 +50,6 @@
         <inertial>
         <origin xyz="0 0 0" rpy="0 0 0" />
-        <mass value="0.05" />
-        <inertia ixx="0.000" ixy="0.0" ixz="0.0" iyy="0.000" iyz="0.0" izz="0.000"/>
+        <mass value="0.005" />
+        <inertia ixx="0.001" ixy="0.0" ixz="0.0" iyy="0.001" iyz="0.0" izz="0.001"/>
         </inertial>
         <visual>
@@ -76,6 +76,6 @@
         <inertial>
         <origin xyz="0.01483 -0.00782 0" rpy="0 0 0" />
-        <mass value="0.05" />
-        <inertia ixx="0.000" ixy="0.0" ixz="0.0" iyy="0.000" iyz="0.0" izz="0.000"/>
+        <mass value="0.002" />
+        <inertia ixx="0.001" ixy="0.0" ixz="0.0" iyy="0.001" iyz="0.0" izz="0.001"/>
         </inertial>
         <visual>
@@ -106,6 +106,6 @@
         <inertial>
         <origin xyz="0.03869 -0.0005 0.00093" rpy="0 0 0" />
-        <mass value="0.05" />
-        <inertia ixx="0.000" ixy="0.0" ixz="0.0" iyy="0.000" iyz="0.0" izz="0.000"/>
+        <mass value="0.001" />
+        <inertia ixx="0.001" ixy="0.001" ixz="0.0" iyy="0.001" iyz="0.0" izz="0.001"/>
         </inertial>
         <visual>
@@ -133,6 +133,6 @@
         <inertial>
         <origin xyz="-0.0153 -0.00602 0" rpy="0 0 0" />
-        <mass value="0.05" />
-        <inertia ixx="0.000" ixy="0.0" ixz="0.0" iyy="0.000" iyz="0.0" izz="0.000"/>
+        <mass value="0.002" />
+        <inertia ixx="0.001" ixy="0.0" ixz="0.0" iyy="0.001" iyz="0.0" izz="0.001"/>
         </inertial>
         <visual>
@@ -161,6 +161,6 @@
         <inertial>
         <origin xyz="-0.01211 -0.00197 0.00093" rpy="0 0 0" />
-        <mass value="0.05" />
-        <inertia ixx="0.000" ixy="0.0" ixz="0.0" iyy="0.00" iyz="0.0" izz="0.00"/>
+        <mass value="0.001" />
+        <inertia ixx="0.001" ixy="0.0" ixz="0.0" iyy="0.001" iyz="0.0" izz="0.001"/>
         </inertial>
         <visual>
@@ -183,9 +183,9 @@
     </joint>
     <!-- SMALL CUBE FOR GRIPPER PLUGIN -->
-    <link name="EE_egp64">
+    <!-- <link name="EE_egp64">
         <inertial>
         <origin xyz="0 0 0" rpy="0 0 0" />
-        <mass value="0.05" />
-        <inertia ixx="0.000" ixy="0.0" ixz="0.0" iyy="0.00" iyz="0.0" izz="0.0"/>
+        <mass value="0.00001" />
+        <inertia ixx="0.001" ixy="0.0" ixz="0.0" iyy="0.001" iyz="0.0" izz="0.001"/>
         </inertial>
         <visual>
@@ -194,11 +194,11 @@
         </geometry>
         </visual>
-    </link>
-    <joint name="EE_egp64_joint" type="fixed" >
+    </link> -->
+    <!-- <joint name="EE_egp64_joint" type="fixed" >
         <parent link="egp64_gripper_base_link" />
         <child link="EE_egp64" />
         <axis xyz="1 0 0" />
         <origin xyz="0.033 -0.018 0.15" rpy="0 0 0"/>
-    </joint>
+    </joint> -->
     <!-- 夹爪传动 -->
     <transmission name="egp64_left_finger_trans">
