Commit message: add pipettle workflow

File: src/abb_gofa_description/urdf/abb_gofa/abb_gofa.urdf.xacro (robot description, xacro)
@@ -36,3 +36,51 @@
       <origin xyz="-0.2 -0.0 0.355" rpy="0.0 0.0 0.0" />
     </joint>
+    <link name="NMR">
+      <visual>
+        <origin xyz="0.0 0.0 0.0" rpy="0.0 0.0 0.0"/>
+        <geometry>
+            <mesh filename="file://$(find abb_gofa_description)/meshes/NMR/NMR.dae"/>
+        </geometry>
+      </visual>
+      <collision>
+        <origin xyz="0.0 0.0 0.0" rpy="0.0 0.0 0.0"/>
+        <geometry>
+            <mesh filename="file://$(find abb_gofa_description)/meshes/NMR/NMR.dae"/>
+        </geometry>
+      </collision>
+      <inertial>
+        <origin xyz="0.0 0.0 0.0" rpy="0.0 0.0 0.0"/>
+        <mass value="50"/>
+        <inertia ixx="0.01" ixy="0.0" ixz="0.0" iyy="0.01" iyz="0.0" izz="0.01"/>
+      </inertial>
+    </link>
+    <joint name="world2NMR" type="fixed">
+      <parent link="world" />
+      <child link = "NMR" />
+      <origin xyz="0.1 -0.8 0.70" rpy="0.0 0.0 -1.570796"/>
+    </joint>
+    <!-- <link name="executor_bracket">
+      <visual>
+        <origin xyz="0.0 0.0 0.0" rpy="0.0 0.0 0.0"/>
+        <geometry>
+            <mesh filename="file://$(find abb_gofa_description)/meshes/executor_bracket/executor_bracket.dae"/>
+        </geometry>
+      </visual>
+      <collision>
+        <origin xyz="0.0 0.0 0.0" rpy="0.0 0.0 0.0"/>
+        <geometry>
+            <mesh filename="file://$(find abb_gofa_description)/meshes/executor_bracket/executor_bracket.dae"/>
+        </geometry>
+      </collision>
+      <inertial>
+        <origin xyz="0.0 0.0 0.0" rpy="0.0 0.0 0.0"/>
+        <mass value="50"/>
+        <inertia ixx="0.01" ixy="0.0" ixz="0.0" iyy="0.01" iyz="0.0" izz="0.01"/>
+      </inertial>
+    </link>
+    <joint name="world2bracket" type="fixed">
+      <parent link="world" />
+      <child link = "executor_bracket" />
+      <origin xyz="-0.6  0.0  0.72" rpy="0.0 0.0 1.570796"/>
+    </joint> -->
 </robot>

File: src/abb_gofa_description/urdf/abb_gofa/abb_gofa_macro.urdf.xacro (robot description, xacro)
@@ -73,22 +73,22 @@
         <link name="link_3">
             <visual>
-            <origin rpy="0.0 0.0 0.0" xyz="0.0 0.0 0.0"/>
-            <geometry>
-                <mesh filename="file://$(find abb_gofa_description)/meshes/abb_gofa/visual/link_3.dae"/>
-            </geometry>
-            <material name="light_grey">
-                <color rgba="0.6 0.6 0.6 1.0"/>
-            </material>
-            </visual>
-            <collision>
-            <origin rpy="0.0 0.0 0.0" xyz="0.0 0.0 0.0"/>
-            <geometry>
-                <mesh filename="file://$(find abb_gofa_description)/meshes/abb_gofa/collision/link_3.dae"/>
-            </geometry>
-            </collision>
-            <inertial>
-            <origin rpy="0.0 0.0 0.0" xyz="0.0 0.0 0.0"/>
-            <mass value="3.4"/>
-            <inertia ixx="0.017" ixy="0.0" ixz="0.0" iyy="0.014" iyz="0.0" izz="0.013"/>
+                <origin rpy="0.0 0.0 0.0" xyz="0.0 0.0 0.0"/>
+                <geometry>
+                    <mesh filename="file://$(find abb_gofa_description)/meshes/abb_gofa/visual/link_3.dae"/>
+                </geometry>
+                <material name="light_grey">
+                    <color rgba="0.6 0.6 0.6 1.0"/>
+                </material>
+            </visual>
+            <collision>
+                <origin rpy="0.0 0.0 0.0" xyz="0.0 0.0 0.0"/>
+                <geometry>
+                    <mesh filename="file://$(find abb_gofa_description)/meshes/abb_gofa/collision/link_3.dae"/>
+                </geometry>
+            </collision>
+            <inertial>
+                <origin rpy="0.0 0.0 0.0" xyz="0.0 0.0 0.0"/>
+                <mass value="3.4"/>
+                <inertia ixx="0.017" ixy="0.0" ixz="0.0" iyy="0.014" iyz="0.0" izz="0.013"/>
             </inertial>
         </link>

File: src/abb_gofa_description/urdf/egp64/egp64.urdf.xacro (robot description, xacro)
@@ -6,5 +6,5 @@
         <inertial>
             <origin xyz="0.0 0.0 0.0" rpy="0.0 0.0 0.0"/>
-            <mass value="0.001" />
+            <mass value="0.01" />
             <inertia ixx="0.001" ixy="0.0" ixz="0.0" iyy="0.001" iyz="0.0" izz="0.001"/>
         </inertial>
@@ -21,6 +21,6 @@
     </link>
     <gazebo reference="connection">
-        <mu1>0.99</mu1>
-        <mu2>0.99</mu2>
+        <mu1>0.8</mu1>
+        <mu2>0.8</mu2>
         <material>Gazebo/Black</material>
     </gazebo>
@@ -43,5 +43,5 @@
         <inertial>
         <origin xyz="0 0 0" rpy="0 0 ${pi/2}" />
-        <mass value="0.001" />
+        <mass value="0.01" />
         <inertia ixx="0.001" ixy="0.0" ixz="0.0" iyy="0.001" iyz="0.0" izz="0.001"/>
         </inertial>

File: src/abb_gofa_description/urdf/pipettle/pipettle.urdf.xacro (robot description, xacro)
@@ -6,7 +6,7 @@
     <link name="pipettle_base">
         <inertial>
-        <mass value="10"/>
+        <mass value="1"/>
         <origin xyz="0 0 0"/>
-        <inertia ixx="100" ixy="0" ixz="0" iyy="100" iyz="0" izz="100"/>
+        <inertia ixx="0.01" ixy="0" ixz="0" iyy="0.01" iyz="0" izz="0.01"/>
         </inertial>
         <visual>
@@ -23,7 +23,7 @@
     <link name="pipettle_link">
         <inertial>
-        <mass value="0.001"/>
+        <mass value="0.0001"/>
         <origin xyz="0 0 0"/>
-        <inertia ixx="0.001" ixy="0" ixz="0" iyy="0.001" iyz="0" izz="0.001"/>
+        <inertia ixx="0.0001" ixy="0" ixz="0" iyy="0.0001" iyz="0" izz="0.0001"/>
         </inertial>
         <visual>
@@ -40,7 +40,7 @@
     <link name="pipettle_clicker">
         <inertial>
-        <mass value="0.001"/>
+        <mass value="0.0001"/>
         <origin xyz="0 0 0"/>
-        <inertia ixx="0.001" ixy="0" ixz="0" iyy="0.001" iyz="0" izz="0.001"/>
+        <inertia ixx="0.0001" ixy="0" ixz="0" iyy="0.0001" iyz="0" izz="0.0001"/>
         </inertial>
         <visual>
@@ -57,7 +57,7 @@
     <link name="pipettle_body">
         <inertial>
-        <mass value="0.001"/>
+        <mass value="0.0001"/>
         <origin xyz="0 0 0"/>
-        <inertia ixx="0.001" ixy="0" ixz="0" iyy="0.001" iyz="0" izz="0.001"/>
+        <inertia ixx="0.0001" ixy="0" ixz="0" iyy="0.0001" iyz="0" izz="0.0001"/>
         </inertial>
         <visual>
@@ -74,7 +74,7 @@
     <link name="pipettle_nib">
         <inertial>
-        <mass value="0.001"/>
+        <mass value="0.0001"/>
         <origin xyz="0 0 0"/>
-        <inertia ixx="0.001" ixy="0" ixz="0" iyy="0.001" iyz="0" izz="0.001"/>
+        <inertia ixx="0.0001" ixy="0" ixz="0" iyy="0.0001" iyz="0" izz="0.0001"/>
         </inertial>
         <visual>
