Commit message: load controller successfully

File: src/abb_gofa_description/urdf/egp64/egp64.urdf.xacro (robot description, xacro)
@@ -2,5 +2,5 @@
 <robot name="egp64" xmlns:xacro="http://www.ros.org/wiki/xacro">
     <xacro:include filename="$(find abb_gofa_description)/urdf/egp64/egp64_ros2_control.urdf.xacro" />
-    <xacro:insert_egp64_ros2_control/>
+    <xacro:egp64_ros2_control/>
     <link name="connection">
         <inertial>

File: src/abb_gofa_description/urdf/egp64/egp64_ros2_control.urdf.xacro (robot description, xacro)
@@ -1,41 +1,32 @@
 <?xml version="1.0"?>
 <robot xmlns:xacro="http://www.ros.org/wiki/xacro">
-    <xacro:macro name="insert_egp64_ros2_control">
-        <xacro:property name="name" value="GazeboSystem" />
+    <xacro:macro name="egp64_ros2_control">
         <gazebo>
-            <plugin name="link_attacher_plugin" filename="liblink_attacher_plugin.so"></plugin>
+            <!-- <plugin name="link_attacher_plugin" filename="liblink_attacher_plugin.so"></plugin> -->
             <plugin filename="libgazebo_ros2_control.so" name="gazebo_ros2_control">
                 <robot_sim_type>gazebo_ros2_control/GazeboSystem</robot_sim_type>
+                <namespace>/egp64</namespace>
                 <parameters>$(find abb_gofa_description)/config/egp64_controller.yaml</parameters>
-                <namespace>/egp64</namespace>
             </plugin>
         </gazebo>
-        <ros2_control name="${name}" type="system">
+        <ros2_control name="egp64_robot" type="system">
             <hardware>
                 <plugin>gazebo_ros2_control/GazeboSystem</plugin>
             </hardware>
             <joint name="egp64_finger_left_joint">
-            <command_interface name="position">
-                <param name="min">-0.01</param>
-                <param name="max">0.04</param>
-            </command_interface>
-            <command_interface name="velocity">
-                <param name="min">-0.2</param>
-                <param name="max">0.2</param>
-            </command_interface>
-            <state_interface name="position"/>
-            <state_interface name="velocity"/>
+                <command_interface name="position">
+                    <param name="min">-0.01</param>
+                    <param name="max">0.04</param>
+                </command_interface>
+                <state_interface name="position"/>
+                <state_interface name="velocity"/>
             </joint>
             <joint name="egp64_finger_right_joint">
-            <command_interface name="position">
-                <param name="min">-0.01</param>
-                <param name="max">0.04</param>
-            </command_interface>
-            <command_interface name="velocity">
-                <param name="min">-0.2</param>
-                <param name="max">0.2</param>
-            </command_interface>
-            <state_interface name="position"/>
-            <state_interface name="velocity"/>
+                <command_interface name="position">
+                    <param name="min">-0.01</param>
+                    <param name="max">0.04</param>
+                </command_interface>
+                <state_interface name="position"/>
+                <state_interface name="velocity"/>
             </joint>
         </ros2_control>

Commit message: add pipettle and openner

File: src/abb_gofa_description/urdf/egp64/egp64.urdf.xacro (robot description, xacro)
@@ -20,4 +20,9 @@
         </collision>
     </link>
+    <gazebo reference="connection">
+        <mu1>0.99</mu1>
+        <mu2>0.99</mu2>
+        <material>Gazebo/Black</material>
+    </gazebo>
     <joint name="connection" type="fixed">
         <parent link="connection"/>
@@ -107,5 +112,5 @@
         <origin xyz="0.03869 -0.0005 0.00093" rpy="0 0 0" />
         <mass value="0.001" />
-        <inertia ixx="0.001" ixy="0.001" ixz="0.0" iyy="0.001" iyz="0.0" izz="0.001"/>
+        <inertia ixx="0.001" ixy="0.00" ixz="0.0" iyy="0.001" iyz="0.0" izz="0.001"/>
         </inertial>
         <visual>

Commit message: fix attach and detach plugin

File: src/abb_gofa_description/urdf/egp64/egp64.urdf.xacro (robot description, xacro)
@@ -6,5 +6,5 @@
         <inertial>
             <origin xyz="0.0 0.0 0.0" rpy="0.0 0.0 0.0"/>
-            <mass value="0.01" />
+            <mass value="0.001" />
             <inertia ixx="0.001" ixy="0.0" ixz="0.0" iyy="0.001" iyz="0.0" izz="0.001"/>
         </inertial>
@@ -20,9 +20,9 @@
         </collision>
     </link>
-    <gazebo reference="connection">
+    <!-- <gazebo reference="connection">
         <mu1>0.8</mu1>
         <mu2>0.8</mu2>
         <material>Gazebo/Black</material>
-    </gazebo>
+    </gazebo> -->
     <joint name="connection" type="fixed">
         <parent link="connection"/>
@@ -43,5 +43,5 @@
         <inertial>
         <origin xyz="0 0 0" rpy="0 0 ${pi/2}" />
-        <mass value="0.01" />
+        <mass value="0.001" />
         <inertia ixx="0.001" ixy="0.0" ixz="0.0" iyy="0.001" iyz="0.0" izz="0.001"/>
         </inertial>
