Commit message: fix executor problems

File: src/abb_gofa_description/urdf/cap_openner/cap_openner.urdf.xacro (robot description, xacro)
@@ -90,5 +90,5 @@
   </link>
   <joint name="world2base" type="fixed">
-    <origin xyz="0.8 0  0.71" rpy="0.0 0.0 1.57079"/>
+    <origin xyz="0.9 0  0.71" rpy="0.0 0.0 1.57079"/>
     <parent link="world"/>
     <child link="openner_base"/>

File: src/abb_gofa_description/urdf/egp64/egp64.urdf.xacro (robot description, xacro)
@@ -102,5 +102,5 @@
         <parent link="egp64_gripper_base_link" />
         <child link="egp64_finger_left_link" />
-        <limit effort="100" lower="-0.01" upper="0.04" velocity="0.2"/>
+        <limit effort="100" lower="-0.04" upper="0.04" velocity="0.2"/>
         <origin xyz="0.01483 -0.00782 0" rpy="0 0 0" />
         <axis xyz="-1 0 0" />
@@ -157,5 +157,5 @@
         <parent link="egp64_gripper_base_link" />
         <child link="egp64_finger_right_link" />
-        <limit effort="100" lower="-0.01" upper="0.04" velocity="0.2"/>
+        <limit effort="100" lower="-0.04" upper="0.04" velocity="0.2"/>
         <origin xyz="-0.0153 -0.00602 0" rpy="0 0 0" />
         <axis xyz="1 0 0" />

File: src/abb_gofa_description/urdf/egp64/egp64_ros2_control.urdf.xacro (robot description, xacro)
@@ -16,5 +16,5 @@
             <joint name="egp64_finger_left_joint">
                 <command_interface name="position">
-                    <param name="min">-0.01</param>
+                    <param name="min">-0.04</param>
                     <param name="max">0.04</param>
                 </command_interface>
@@ -24,5 +24,5 @@
             <joint name="egp64_finger_right_joint">
                 <command_interface name="position">
-                    <param name="min">-0.01</param>
+                    <param name="min">-0.04</param>
                     <param name="max">0.04</param>
                 </command_interface>
