Commit message: add move_arm_cartesian

File: src/abb_gofa_description/urdf/pipettle/pipettle.urdf.xacro (robot description, xacro)
@@ -6,7 +6,7 @@
     <link name="pipettle_base">
         <inertial>
-        <mass value="1"/>
+        <mass value="2"/>
         <origin xyz="0 0 0"/>
-        <inertia ixx="0.01" ixy="0" ixz="0" iyy="0.01" iyz="0" izz="0.01"/>
+        <inertia ixx="0.05" ixy="0" ixz="0" iyy="0.05" iyz="0" izz="0.05"/>
         </inertial>
         <visual>

Commit message: complete pipettle

File: src/abb_gofa_description/urdf/pipettle/pipettle.urdf.xacro (robot description, xacro)
@@ -6,7 +6,7 @@
     <link name="pipettle_base">
         <inertial>
-        <mass value="2"/>
+        <mass value="1"/>
         <origin xyz="0 0 0"/>
-        <inertia ixx="0.05" ixy="0" ixz="0" iyy="0.05" iyz="0" izz="0.05"/>
+        <inertia ixx="1" ixy="0" ixz="0.00" iyy="1" iyz="0" izz="1"/>
         </inertial>
         <visual>
@@ -23,7 +23,7 @@
     <link name="pipettle_link">
         <inertial>
-        <mass value="0.0001"/>
+        <mass value="0.01"/>
         <origin xyz="0 0 0"/>
-        <inertia ixx="0.0001" ixy="0" ixz="0" iyy="0.0001" iyz="0" izz="0.0001"/>
+        <inertia ixx="0.01" ixy="0" ixz="0" iyy="0.01" iyz="0" izz="0.01"/>
         </inertial>
         <visual>
@@ -40,7 +40,7 @@
     <link name="pipettle_clicker">
         <inertial>
-        <mass value="0.0001"/>
+        <mass value="0.01"/>
         <origin xyz="0 0 0"/>
-        <inertia ixx="0.0001" ixy="0" ixz="0" iyy="0.0001" iyz="0" izz="0.0001"/>
+        <inertia ixx="0.01" ixy="0" ixz="0" iyy="0.01" iyz="0" izz="0.01"/>
         </inertial>
         <visual>
@@ -57,7 +57,7 @@
     <link name="pipettle_body">
         <inertial>
-        <mass value="0.0001"/>
+        <mass value="0.01"/>
         <origin xyz="0 0 0"/>
-        <inertia ixx="0.0001" ixy="0" ixz="0" iyy="0.0001" iyz="0" izz="0.0001"/>
+        <inertia ixx="0.01" ixy="0" ixz="0" iyy="0001" iyz="0" izz="0.01"/>
         </inertial>
         <visual>
@@ -74,7 +74,7 @@
     <link name="pipettle_nib">
         <inertial>
-        <mass value="0.0001"/>
+        <mass value="0.01"/>
         <origin xyz="0 0 0"/>
-        <inertia ixx="0.0001" ixy="0" ixz="0" iyy="0.0001" iyz="0" izz="0.0001"/>
+        <inertia ixx="0.01" ixy="0" ixz="0" iyy="0.01" iyz="0" izz="0.01"/>
         </inertial>
         <visual>
